Commit message: [HOTFIX] hector_v1 torso name fix

File: source/hector_v1/mvsc_reduced.urdf (robot description, URDF)
Before this commit: robot w_coupling, 19 links, 18 joints
Links:
- removed link hector_v1p5
- added link torso, mass 1.0; collision mesh filename=meshes/base_visuals.obj scale=1. 1. 1.; visual mesh filename=meshes/base_visuals.obj scale=1. 1. 1.
Joints:
- joint l_hip_yaw_joint: parent hector_v1p5 -> torso
- joint r_hip_yaw_joint: parent hector_v1p5 -> torso
