Commit message: Update mvsc_reduced.urdf
Uncommented the visual block for hip_roll link/motor

File: source/hector_v2/feet/mvsc_reduced.urdf (robot description, URDF)
Before this commit: robot mvmc_reduced, 19 links, 18 joints
Links:
- link l_hip1: geometry collision cylinder length=0.044 radius=0.0465; visual mesh filename=../meshes/l_hip1.stl scale=1.00000 1.00000 1.00000
