Commit message: moved into source

File: source/hector_v2/feet/mvmc_reduced.urdf (robot description, URDF)
Before this commit: robot hector_v2, 19 links, 18 joints
Links:
- link l_calf: geometry collision mesh filename=../meshes/calf.stl scale=1.00000 1.00000 1.00000; visual mesh filename=../meshes/calf.stl scale=1.00000 1.00000 1.00000
- link l_hip1: geometry collision mesh filename=../meshes/l_hip1.stl scale=1.00000 1.00000 1.00000; visual mesh filename=../meshes/l_hip1.stl scale=1.00000 1.00000 1.00000
- link l_hip2: geometry collision mesh filename=../meshes/l_hip2.stl scale=1.00000 1.00000 1.00000; visual mesh filename=../meshes/l_hip2.stl scale=1.00000 1.00000 1.00000
- link l_lower_arm: geometry collision mesh filename=../meshes/lower_arm.stl scale=1.00000 1.00000 1.00000; visual mesh filename=../meshes/lower_arm.stl scale=1.00000 1.00000 1.00000
- link l_shoudler1: geometry collision mesh filename=../meshes/l_shoulder1.stl scale=1.00000 1.00000 1.00000; visual mesh filename=../meshes/l_shoulder1.stl scale=1.00000 1.00000 1.00000
- link l_shoulder2: geometry collision mesh filename=../meshes/l_shoulder2.stl scale=1.00000 1.00000 1.00000; visual mesh filename=../meshes/l_shoulder2.stl scale=1.00000 1.00000 1.00000
- link l_thigh: geometry collision mesh filename=../meshes/l_thigh.stl scale=1.00000 1.00000 1.00000; visual mesh filename=../meshes/l_thigh.stl scale=1.00000 1.00000 1.00000
- link l_toe: geometry collision mesh filename=../meshes/foot.stl scale=1.00000 1.00000 1.00000; visual mesh filename=../meshes/foot.stl scale=1.00000 1.00000 1.00000
- link l_upper_arm: geometry collision mesh filename=../meshes/l_upper_arm.stl scale=1.00000 1.00000 1.00000; visual mesh filename=../meshes/l_upper_arm.stl scale=1.00000 1.00000 1.00000
- link r_calf: geometry collision mesh filename=../meshes/calf.stl scale=1.00000 1.00000 1.00000; visual mesh filename=../meshes/calf.stl scale=1.00000 1.00000 1.00000
- link r_hip1: geometry collision mesh filename=../meshes/r_hip1.stl scale=1.00000 1.00000 1.00000; visual mesh filename=../meshes/r_hip1.stl scale=1.00000 1.00000 1.00000
- link r_hip2: geometry collision mesh filename=../meshes/r_hip2.stl scale=1.00000 1.00000 1.00000; visual mesh filename=../meshes/r_hip2.stl scale=1.00000 1.00000 1.00000
- link r_lower_arm: geometry collision mesh filename=../meshes/lower_arm.stl scale=1.00000 1.00000 1.00000; visual mesh filename=../meshes/lower_arm.stl scale=1.00000 1.00000 1.00000
- link r_shoulder1: geometry collision mesh filename=../meshes/r_shoulder1.stl scale=1.00000 1.00000 1.00000; visual mesh filename=../meshes/r_shoulder1.stl scale=1.00000 1.00000 1.00000
- link r_shoulder2: geometry collision mesh filename=../meshes/r_shoulder2.stl scale=1.00000 1.00000 1.00000; visual mesh filename=../meshes/r_shoulder2.stl scale=1.00000 1.00000 1.00000
- link r_thigh: geometry collision mesh filename=../meshes/r_thigh.stl scale=1.00000 1.00000 1.00000; visual mesh filename=../meshes/r_thigh.stl scale=1.00000 1.00000 1.00000
- link r_toe: geometry collision mesh filename=../meshes/foot.stl scale=1.00000 1.00000 1.00000; visual mesh filename=../meshes/foot.stl scale=1.00000 1.00000 1.00000
- link r_upper_arm: geometry collision mesh filename=../meshes/r_upper_arm.stl scale=1.00000 1.00000 1.00000; visual mesh filename=../meshes/r_upper_arm.stl scale=1.00000 1.00000 1.00000
- link torso: geometry collision mesh filename=../meshes/torso.stl scale=1.00000 1.00000 1.00000; visual mesh filename=../meshes/torso.stl scale=1.00000 1.00000 1.00000

Commit message: [HOTFIX] exposes constants  and adds bad_contact_bodies

File: source/hector_v2/feet/mvmc_reduced.urdf (robot description, URDF)
Before this commit: robot hector_v2, 19 links, 18 joints
Links:
- removed link l_shoudler1
- added link l_shoulder1, mass 0.43560; collision mesh filename=../meshes/l_shoulder1.stl scale=1.00000 1.00000 1.00000; visual mesh filename=../meshes/l_shoulder1.stl scale=1.00000 1.00000 1.00000
Joints:
- joint l_shoulder_pitch: parent l_shoudler1 -> l_shoulder1
- joint l_shoulder_yaw: child l_shoudler1 -> l_shoulder1

Commit message: hector_v2 ee added, tbt

File: source/hector_v2/feet/mvmc_reduced.urdf (robot description, URDF)
Before this commit: robot mvmc_reduced, 19 links, 18 joints
Links:
- added link l_hand
- added link r_hand
Joints:
- added joint l_wrist: type fixed, parent l_lower_arm, child l_hand, origin xyz=0 0 -0.23 rpy=0 0 0
- added joint r_wrist: type fixed, parent r_lower_arm, child r_hand, origin xyz=0 0 -0.23 rpy=0 0 0

Commit message: hector_v2 ee add, tested

File: source/hector_v2/feet/mvmc_reduced.urdf (robot description, URDF)
Before this commit: robot mvmc_reduced, 21 links, 20 joints
Links:
- link l_hand: mass None -> 0.001
- link r_hand: mass None -> 0.001

Commit message: defines end effector chains (#23)
* ee added for g1, motion_1

* digit ee added

* hector_v2 ee added, tbt

* hector_v2 ee add, tested

* added joint chains for ee

* add links_in_chain for humanoids

File: source/hector_v2/feet/mvmc_reduced.urdf (robot description, URDF)
Before this commit: robot mvmc_reduced, 19 links, 18 joints
Links:
- added link l_hand, mass 0.001
- added link r_hand, mass 0.001
Joints:
- added joint l_wrist: type fixed, parent l_lower_arm, child l_hand, origin xyz=0 0 -0.23 rpy=0 0 0
- added joint r_wrist: type fixed, parent r_lower_arm, child r_hand, origin xyz=0 0 -0.23 rpy=0 0 0

Commit message: Changed joint limit, realign between xml and urdf, updated elbow gear ratio

File: source/hector_v2/feet/mvmc_reduced.urdf (robot description, URDF)
Before this commit: robot mvmc_reduced, 21 links, 20 joints
Joints:
- joint l_elbow: limit lower=-1.5708 upper=1.5708 effort=17.0 velocity=32.0 -> lower=-2.5 upper=2.5 effort=17.0 velocity=32.0
- joint l_shoulder_pitch: limit lower=-1.5708 upper=1.5708 effort=17.0 velocity=32.0 -> lower=-3.14 upper=3.14 effort=17.0 velocity=32.0
- joint l_shoulder_roll: limit lower=-1.5708 upper=1.5708 effort=17.0 velocity=32.0 -> lower=-1.4 upper=1.4 effort=17.0 velocity=32.0
- joint r_elbow: limit lower=-1.5708 upper=1.5708 effort=17.0 velocity=32.0 -> lower=-2.5 upper=2.5 effort=17.0 velocity=32.0
- joint r_shoulder_pitch: limit lower=-1.5708 upper=1.5708 effort=17.0 velocity=32.0 -> lower=-3.14 upper=3.14 effort=17.0 velocity=32.0
- joint r_shoulder_roll: limit lower=-1.5708 upper=1.5708 effort=17.0 velocity=32.0 -> lower=-1.4 upper=1.4 effort=17.0 velocity=32.0

File: source/hector_v2/feet/mvsc_reduced.urdf (robot description, URDF)
Before this commit: robot mvmc_reduced, 19 links, 18 joints
Joints:
- joint l_elbow: limit lower=-1.5708 upper=1.5708 effort=17.0 velocity=32.0 -> lower=-2.5 upper=2.5 effort=17.0 velocity=32.0
- joint l_shoulder_pitch: limit lower=-1.5708 upper=1.5708 effort=17.0 velocity=32.0 -> lower=-3.14 upper=3.14 effort=17.0 velocity=32.0
- joint l_shoulder_roll: limit lower=-1.5708 upper=1.5708 effort=17.0 velocity=32.0 -> lower=-1.4 upper=1.4 effort=17.0 velocity=32.0
- joint r_elbow: limit lower=-1.5708 upper=1.5708 effort=17.0 velocity=32.0 -> lower=-2.5 upper=2.5 effort=17.0 velocity=32.0
- joint r_shoulder_pitch: limit lower=-1.5708 upper=1.5708 effort=17.0 velocity=32.0 -> lower=-3.14 upper=3.14 effort=17.0 velocity=32.0
- joint r_shoulder_roll: limit lower=-1.5708 upper=1.5708 effort=17.0 velocity=32.0 -> lower=-1.4 upper=1.4 effort=17.0 velocity=32.0
