Commit message: Fixed thighs for hector_v2 simplified collision model and created urdf for tracks

File: source/hector_v2/track/mvsc_track.urdf (robot description, URDF)
Before this commit: robot mvmc_reduced, 19 links, 18 joints
Links:
- added link l_back_wheel, mass 0.001; collision cylinder length=0.02 radius=0.02; visual cylinder length=0.02 radius=0.02
- added link l_front_wheel, mass 0.001; collision cylinder length=0.02 radius=0.02; visual cylinder length=0.02 radius=0.02
- added link r_back_wheel, mass 0.001; collision cylinder length=0.02 radius=0.02; visual cylinder length=0.02 radius=0.02
- added link r_front_wheel, mass 0.001; collision cylinder length=0.02 radius=0.02; visual cylinder length=0.02 radius=0.02
Joints:
- added joint l_toe_back: type continuous, parent l_toe, child l_back_wheel, origin xyz=-0.055 0.0000 -0.0625 rpy=-0.00000 -0.00000 0.00000, axis 0.00000 1.00000 0.00000, limit effort=5.5 velocity=50.0
- added joint l_toe_front: type continuous, parent l_toe, child l_front_wheel, origin xyz=0.0750 0.0000 -0.0625 rpy=-0.00000 -0.00000 0.00000, axis 0.00000 1.00000 0.00000, limit effort=5.5 velocity=50.0
- added joint r_toe_back: type continuous, parent r_toe, child r_back_wheel, origin xyz=-0.055 0.0000 -0.0625 rpy=-0.00000 -0.00000 0.00000, axis 0.00000 1.00000 0.00000, limit effort=5.5 velocity=50.0
- added joint r_toe_front: type continuous, parent r_toe, child r_front_wheel, origin xyz=0.0750 0.0000 -0.0625 rpy=-0.00000 -0.00000 0.00000, axis 0.00000 1.00000 0.00000, limit effort=5.5 velocity=50.0

Commit message: fixed wheel_ and motor velocitie_
my key between wadx on laptop broke

File: source/hector_v2/track/mvsc_track.urdf (robot description, URDF)
Before this commit: robot mvmc_reduced, 23 links, 22 joints
Links:
- link l_back_wheel: geometry collision cylinder length=0.02 radius=0.03; visual cylinder length=0.02 radius=0.03
- link l_front_wheel: geometry collision cylinder length=0.02 radius=0.03; visual cylinder length=0.02 radius=0.03
- link r_back_wheel: geometry collision cylinder length=0.02 radius=0.03; visual cylinder length=0.02 radius=0.03
- link r_front_wheel: geometry collision cylinder length=0.02 radius=0.03; visual cylinder length=0.02 radius=0.03
Joints:
- joint l_toe_back: limit effort=5.5 velocity=50.0 -> effort=5.5 velocity=33.0; origin xyz=-0.055 0.0000 -0.0625 rpy=-0.00000 -0.00000 0.00000 -> xyz=-0.055 0.0000 -0.0725 rpy=-0.00000 -0.00000 0.00000
- joint l_toe_front: limit effort=5.5 velocity=50.0 -> effort=5.5 velocity=33.0; origin xyz=0.0750 0.0000 -0.0625 rpy=-0.00000 -0.00000 0.00000 -> xyz=0.0750 0.0000 -0.0725 rpy=-0.00000 -0.00000 0.00000
- joint r_toe_back: limit effort=5.5 velocity=50.0 -> effort=5.5 velocity=33.0; origin xyz=-0.055 0.0000 -0.0625 rpy=-0.00000 -0.00000 0.00000 -> xyz=-0.055 0.0000 -0.0725 rpy=-0.00000 -0.00000 0.00000
- joint r_toe_front: limit effort=5.5 velocity=50.0 -> effort=5.5 velocity=33.0; origin xyz=0.0750 0.0000 -0.0625 rpy=-0.00000 -0.00000 0.00000 -> xyz=0.0750 0.0000 -0.0725 rpy=-0.00000 -0.00000 0.00000

Commit message: fixed thighs for hector_v2 mvsc and created urdf for track (#31)
* Fixed thighs for hector_v2 simplified collision model and created urdf for tracks

* fixed wheel_ and motor velocitie_

my key between wadx on laptop broke

File: source/hector_v2/track/mvsc_track.urdf (robot description, URDF)
Before this commit: robot mvmc_reduced, 19 links, 18 joints
Links:
- added link l_back_wheel, mass 0.001; collision cylinder length=0.02 radius=0.03; visual cylinder length=0.02 radius=0.03
- added link l_front_wheel, mass 0.001; collision cylinder length=0.02 radius=0.03; visual cylinder length=0.02 radius=0.03
- added link r_back_wheel, mass 0.001; collision cylinder length=0.02 radius=0.03; visual cylinder length=0.02 radius=0.03
- added link r_front_wheel, mass 0.001; collision cylinder length=0.02 radius=0.03; visual cylinder length=0.02 radius=0.03
Joints:
- added joint l_toe_back: type continuous, parent l_toe, child l_back_wheel, origin xyz=-0.055 0.0000 -0.0725 rpy=-0.00000 -0.00000 0.00000, axis 0.00000 1.00000 0.00000, limit effort=5.5 velocity=33.0
- added joint l_toe_front: type continuous, parent l_toe, child l_front_wheel, origin xyz=0.0750 0.0000 -0.0725 rpy=-0.00000 -0.00000 0.00000, axis 0.00000 1.00000 0.00000, limit effort=5.5 velocity=33.0
- added joint r_toe_back: type continuous, parent r_toe, child r_back_wheel, origin xyz=-0.055 0.0000 -0.0725 rpy=-0.00000 -0.00000 0.00000, axis 0.00000 1.00000 0.00000, limit effort=5.5 velocity=33.0
- added joint r_toe_front: type continuous, parent r_toe, child r_front_wheel, origin xyz=0.0750 0.0000 -0.0725 rpy=-0.00000 -0.00000 0.00000, axis 0.00000 1.00000 0.00000, limit effort=5.5 velocity=33.0
