Commit message: updated joint encoder to actuator encoder in xml

File: source/motion_1/m1A_1v5_23dof_FixArm_Updated.urdf (robot description, URDF)
Before this commit: robot motion1_23dof, 27 links, 26 joints
Links:
- link right_ankle_pitch_link: mass 0.077117 -> 0.0771174
- link right_ankle_roll_link: mass 0.716628 -> 0.716625
- link right_knee_link: mass 1.58691 -> 1.58249
