Commit message: Tested the configuration file, fixed broken motion1 config

File: source/motion_1/m1A_1v5_23dof_FixArm.urdf (robot description, URDF)
Before this commit: robot motion1_23dof, 27 links, 26 joints
Links:
- link head_link: geometry visual mesh filename=meshes_reduce/head_link.STL
- link left_ankle_pitch_link: geometry visual mesh filename=meshes_reduce/left_ankle_pitch_link.STL
- link left_ankle_roll_link: geometry collision mesh filename=meshes_reduce/left_ankle_roll_link.STL; visual mesh filename=meshes_reduce/left_ankle_roll_link.STL
- link left_elbow_link: geometry visual mesh filename=meshes_reduce/left_elbow_link.STL
- link left_fist_link: geometry collision mesh filename=meshes_reduce/left_fist_link.STL; visual mesh filename=meshes_reduce/left_fist_link.STL
- link left_hip_pitch_link: geometry visual mesh filename=meshes_reduce/left_hip_pitch_link.STL
- link left_hip_roll_link: geometry visual mesh filename=meshes_reduce/left_hip_roll_link.STL
- link left_hip_yaw_link: geometry visual mesh filename=meshes_reduce/left_hip_yaw_link.STL
- link left_knee_link: geometry visual mesh filename=meshes_reduce/left_knee_link.STL
- link left_shoulder_pitch_link: geometry visual mesh filename=meshes_reduce/left_shoulder_pitch_link.STL
- link left_shoulder_roll_link: geometry visual mesh filename=meshes_reduce/left_shoulder_roll_link.STL
- link left_shoulder_yaw_link: geometry visual mesh filename=meshes_reduce/left_shoulder_yaw_link.STL
- link left_wrist_link: geometry visual mesh filename=meshes_reduce/left_wrist_link.STL
- link pelvis_link: geometry visual mesh filename=meshes_reduce/pelvis_link.STL
- link right_ankle_pitch_link: geometry visual mesh filename=meshes_reduce/right_ankle_pitch_link.STL
- link right_ankle_roll_link: geometry collision mesh filename=meshes_reduce/right_ankle_roll_link.STL; visual mesh filename=meshes_reduce/right_ankle_roll_link.STL
- link right_elbow_link: geometry visual mesh filename=meshes_reduce/right_elbow_link.STL
- link right_fist_link: geometry collision mesh filename=meshes_reduce/right_fist_link.STL; visual mesh filename=meshes_reduce/right_fist_link.STL
- link right_hip_pitch_link: geometry visual mesh filename=meshes_reduce/right_hip_pitch_link.STL
- link right_hip_roll_link: geometry visual mesh filename=meshes_reduce/right_hip_roll_link.STL
- link right_hip_yaw_link: geometry visual mesh filename=meshes_reduce/right_hip_yaw_link.STL
- link right_knee_link: geometry visual mesh filename=meshes_reduce/right_knee_link.STL
- link right_shoulder_pitch_link: geometry visual mesh filename=meshes_reduce/right_shoulder_pitch_link.STL
- link right_shoulder_roll_link: geometry visual mesh filename=meshes_reduce/right_shoulder_roll_link.STL
- link right_shoulder_yaw_link: geometry visual mesh filename=meshes_reduce/right_shoulder_yaw_link.STL
- link right_wrist_link: geometry visual mesh filename=meshes_reduce/right_wrist_link.STL
- link torso_link: geometry collision mesh filename=meshes_reduce/torso_link.STL; visual mesh filename=meshes_reduce/torso_link.STL
Joints:
- removed joint left_wrist_joint
- removed joint right_wrist_joint
- removed joint waist_joint
- added joint left_wrist_roll_joint: type revolute, parent left_elbow_link, child left_wrist_link, origin xyz=0 0 -0.09 rpy=0 0 0, axis 0 0 1, limit lower=-3.1 upper=3.1 effort=17 velocity=42.9
- added joint right_wrist_roll_joint: type revolute, parent right_elbow_link, child right_wrist_link, origin xyz=0 0 -0.09 rpy=0 0 0, axis 0 0 1, limit lower=-3.1 upper=3.1 effort=17 velocity=42.9
- added joint waist_yaw_joint: type revolute, parent torso_link, child pelvis_link, origin xyz=0 0 -0.181 rpy=0 0 0, axis 0 0 1, limit lower=-1.57 upper=1.57 effort=60 velocity=20.4
- joint left_fist_joint: limit lower=-1.5 upper=1.5 effort=17 velocity=42.9 -> (none); type revolute -> fixed
- joint right_fist_joint: limit lower=-1.5 upper=1.5 effort=17 velocity=42.9 -> (none); type revolute -> fixed

Commit message: changed wrist_roll to wrist_yaw

File: source/motion_1/m1A_1v5_23dof_FixArm.urdf (robot description, URDF)
Before this commit: robot motion1_23dof, 27 links, 26 joints
Joints:
- removed joint left_wrist_roll_joint
- removed joint right_wrist_roll_joint
- added joint left_wrist_yaw_joint: type revolute, parent left_elbow_link, child left_wrist_link, origin xyz=0 0 -0.09 rpy=0 0 0, axis 0 0 1, limit lower=-3.1 upper=3.1 effort=17 velocity=42.9
- added joint right_wrist_yaw_joint: type revolute, parent right_elbow_link, child right_wrist_link, origin xyz=0 0 -0.09 rpy=0 0 0, axis 0 0 1, limit lower=-3.1 upper=3.1 effort=17 velocity=42.9

File: source/motion_1/mvsc.urdf (robot description, URDF)
Before this commit: robot motion1_23dof, 27 links, 26 joints
Joints:
- removed joint left_wrist_roll_joint
- removed joint right_wrist_roll_joint
- added joint left_wrist_yaw_joint: type revolute, parent left_elbow_link, child left_wrist_link, origin xyz=0 0 -0.09 rpy=0 0 0, axis 0 0 1, limit lower=-3.1 upper=3.1 effort=17 velocity=42.9
- added joint right_wrist_yaw_joint: type revolute, parent right_elbow_link, child right_wrist_link, origin xyz=0 0 -0.09 rpy=0 0 0, axis 0 0 1, limit lower=-3.1 upper=3.1 effort=17 velocity=42.9

Commit message: delete old urdf

File: source/motion_1/m1A_1v5_23dof_FixArm.urdf (robot description, URDF)
Before this commit: robot motion1_23dof, 27 links, 26 joints
Links:
- link right_ankle_pitch_link: mass 0.077117 -> 0.0771174
- link right_ankle_roll_link: mass 0.716628 -> 0.716625
- link right_knee_link: mass 1.58691 -> 1.58249
Joints:
- joint left_shoulder_pitch_joint: origin xyz=0 0.103122 0.121183 rpy=0.17453289056207222 0.0 0.0 -> xyz=0 0.103122 0.302183 rpy=0.17453289056207222 0.0 0.0
- joint neck_joint: origin xyz=0 0 0.181 rpy=0 0 0 -> xyz=0 0 0.362 rpy=0 0 0
- joint right_shoulder_pitch_joint: origin xyz=0 -0.103122 0.121183 rpy=-0.17453289056207222 0.0 0.0 -> xyz=0 -0.103122 0.302183 rpy=-0.17453289056207222 0.0 0.0
- joint waist_yaw_joint: child pelvis_link -> torso_link; origin xyz=0 0 -0.181 rpy=0 0 0 -> xyz=0 0 0 rpy=0 0 0; parent torso_link -> pelvis_link
