Commit message: [HOTFIX]commented out minipi calf collision

File: source/mini_pi/pi_12dof_release_v1.urdf (robot description, URDF)
Before this commit: robot pi_12dof_release_v1, 13 links, 12 joints
Links:
- link l_ankle_pitch_link: geometry visual mesh filename=meshes/l_ankle_pitch_link.STL
- link l_calf_link: geometry visual mesh filename=meshes/l_calf_link.STL
- link r_ankle_pitch_link: geometry visual mesh filename=meshes/r_ankle_pitch_link.STL
- link r_calf_link: geometry visual mesh filename=meshes/r_calf_link.STL

Commit message: decimate meshes, changed 0 angle pos, changed default_joint_pos

File: source/mini_pi/pi_12dof_release_v1.urdf (robot description, URDF)
Before this commit: robot pi_12dof_release_v1, 13 links, 12 joints
Joints:
- joint l_ankle_pitch_joint: origin xyz=0 0 -0.14 rpy=0 -0.4 0 -> xyz=0 0 -0.14 rpy=0 0 0
- joint l_calf_joint: origin xyz=0 0 -0.07025 rpy=0 0.65 0 -> xyz=0 0 -0.07025 rpy=0 0 0
- joint l_hip_pitch_joint: origin xyz=-5.1979E-05 0.0233 -0.033 rpy=0 -0.25 0 -> xyz=-5.1979E-05 0.0233 -0.033 rpy=0 0 0
- joint r_ankle_pitch_joint: origin xyz=0 0 -0.14 rpy=0 -0.4 0 -> xyz=0 0 -0.14 rpy=0 0 0
- joint r_calf_joint: origin xyz=0 -0.0027 -0.07025 rpy=0 0.65 0 -> xyz=0 -0.0027 -0.07025 rpy=0 0 0
- joint r_hip_pitch_joint: origin xyz=-5.1979E-05 -0.0233 -0.033 rpy=0 -0.25 0 -> xyz=-5.1979E-05 -0.0233 -0.033 rpy=0 0 0
