Commit message: Update mass of thighs to match v5

File: source/hector_mini/mvmc.urdf (robot description, URDF)
Before this commit: robot hector_mini, 13 links, 12 joints
Links:
- link left_hip_pitch_joint: mass 0.9856 -> 0.5
- link right_hip_pitch_joint: mass 0.9856 -> 0.5

Commit message: Fixed mass of motors for thigh assem

File: source/hector_mini/mvmc.urdf (robot description, URDF)
Before this commit: robot hector_mini, 13 links, 12 joints
Links:
- link left_hip_pitch_joint: mass 0.5 -> 1.084915
- link right_hip_pitch_joint: mass 0.5 -> 1.084915

Commit message: Update inertial properties of hector-mini thighs and calves to match v5 (#48)
* Update inertial properties for calf links

* Update inertial properties for thigh joints

* Update inertial properties for thighs/calves

* Update thigh/calf to match v5

* Update mass of thighs to match v5

* Fixed mass of motors for thigh assem

* Fixed mass of motors for thigh assem

File: source/hector_mini/mvmc.urdf (robot description, URDF)
Before this commit: robot hector_mini, 13 links, 12 joints
Links:
- link left_hip_pitch_joint: mass 0.9856 -> 1.084915
- link right_hip_pitch_joint: mass 0.9856 -> 1.084915
