Commit message: Added d435 urdf link, copied from unitree 'g1_29dof_rev_1_0 urdf'

File: source/g1/g1_bm.urdf (robot description, URDF)
Before this commit: robot g1, 40 links, 39 joints
Links:
- added link d435_link
Joints:
- added joint d435_joint: type fixed, parent torso_link, child d435_link, origin xyz=0.0576235 0.01753 0.42987 rpy=0 0.8307767239493009 0
