Commit message: added accurate flat hand collision, added extra no weight body for force application

File: source/g1/g1_flat_0_hand.urdf (robot description, URDF)
Before this commit: robot g1, 41 links, 40 joints
Links:
- added link left_force_applicator_link, mass 0.001
- added link right_force_applicator_link, mass 0.001
- link left_rubber_hand: geometry collision mesh filename=meshes/left_flat_hand.stl; visual mesh filename=meshes/left_flat_hand.stl
- link left_wrist_yaw_link: geometry collision mesh filename=meshes/left_wrist_yaw_link.STL; visual mesh filename=meshes/left_wrist_yaw_link.STL
- link right_rubber_hand: geometry collision mesh filename=meshes/right_flat_hand.stl; visual mesh filename=meshes/right_flat_hand.stl
- link right_wrist_yaw_link: geometry collision mesh filename=meshes/right_wrist_yaw_link.STL; visual mesh filename=meshes/right_wrist_yaw_link.STL
Joints:
- added joint left_force_applicator: type fixed, parent left_wrist_yaw_link, child left_force_applicator_link, origin xyz=0.12 0 0 rpy=0 0 0
- added joint right_force_applicator: type fixed, parent right_wrist_yaw_link, child right_force_applicator_link, origin xyz=0.12 0 0 rpy=0 0 0

Commit message: custom patch collision, remove wrist yaw collision

File: source/g1/g1_flat_0_hand.urdf (robot description, URDF)
Before this commit: robot g1, 43 links, 42 joints
Links:
- link left_force_applicator_link: geometry collision box size=0.14 -0.01 0.09
- link left_rubber_hand: geometry visual mesh filename=meshes/left_flat_hand.stl
- link left_wrist_yaw_link: geometry visual mesh filename=meshes/left_wrist_yaw_link.STL
- link right_force_applicator_link: geometry collision box size=0.14 0.01 0.09
- link right_rubber_hand: geometry visual mesh filename=meshes/right_flat_hand.stl
- link right_wrist_yaw_link: geometry visual mesh filename=meshes/right_wrist_yaw_link.STL
Joints:
- joint left_force_applicator: origin xyz=0.12 0 0 rpy=0 0 0 -> xyz=0.12 -0.01 0 rpy=0 0 0
- joint right_force_applicator: origin xyz=0.12 0 0 rpy=0 0 0 -> xyz=0.12 0.01 0 rpy=0 0 0

Commit message: fixed box dimension

File: source/g1/g1_flat_0_hand.urdf (robot description, URDF)
Before this commit: robot g1, 43 links, 42 joints
Links:
- link left_force_applicator_link: geometry collision box size=0.14 0.01 0.09

Commit message: Jm/flat hand simplified (#55)
* custom patch collision, remove wrist yaw collision

* fixed box dimension

File: source/g1/g1_flat_0_hand.urdf (robot description, URDF)
Before this commit: robot g1, 43 links, 42 joints
Links:
- link left_force_applicator_link: geometry collision box size=0.14 0.01 0.09
- link left_rubber_hand: geometry visual mesh filename=meshes/left_flat_hand.stl
- link left_wrist_yaw_link: geometry visual mesh filename=meshes/left_wrist_yaw_link.STL
- link right_force_applicator_link: geometry collision box size=0.14 0.01 0.09
- link right_rubber_hand: geometry visual mesh filename=meshes/right_flat_hand.stl
- link right_wrist_yaw_link: geometry visual mesh filename=meshes/right_wrist_yaw_link.STL
Joints:
- joint left_force_applicator: origin xyz=0.12 0 0 rpy=0 0 0 -> xyz=0.12 -0.01 0 rpy=0 0 0
- joint right_force_applicator: origin xyz=0.12 0 0 rpy=0 0 0 -> xyz=0.12 0.01 0 rpy=0 0 0
