Commit message: fixed largebox and add semantic tags

File: source/omomo_objects/largebox/largebox.urdf (robot description, URDF)
Before this commit: robot largebox, 1 links, 0 joints
Links:
- removed link largebox_link
- added link base_link, mass 1.00000; collision mesh filename=largebox.obj; visual mesh filename=largebox.obj
