Commit message: Update mass properties for OMOMO URDF objects

File: source/omomo_objects/clothesstand/clothesstand.urdf (robot description, URDF)
Before this commit: robot clothesstand, 1 links, 0 joints
Links:
- link base_link: mass 1.00000 -> 1.50000

File: source/omomo_objects/largebox/largebox.urdf (robot description, URDF)
Before this commit: robot largebox, 1 links, 0 joints
Links:
- link base_link: mass 1.00000 -> 4.50000

File: source/omomo_objects/largetable/largetable.urdf (robot description, URDF)
Before this commit: robot largetable, 1 links, 0 joints
Links:
- link base_link: mass 1.00000 -> 4.50000

File: source/omomo_objects/monitor/monitor.urdf (robot description, URDF)
Before this commit: robot monitor, 1 links, 0 joints
Links:
- link base_link: mass 1.00000 -> 2.00000

File: source/omomo_objects/plasticbox/plasticbox.urdf (robot description, URDF)
Before this commit: robot plasticbox, 1 links, 0 joints
Links:
- link base_link: mass 1.00000 -> 1.50000

File: source/omomo_objects/smallbox/smallbox.urdf (robot description, URDF)
Before this commit: robot smallbox, 1 links, 0 joints
Links:
- link base_link: mass 1.00000 -> 0.80000

File: source/omomo_objects/suitcase/suitcase.urdf (robot description, URDF)
Before this commit: robot suitcase, 1 links, 0 joints
Links:
- link base_link: mass 1.00000 -> 2.00000

File: source/omomo_objects/trashcan/trashcan.urdf (robot description, URDF)
Before this commit: robot trashcan, 1 links, 0 joints
Links:
- link base_link: mass 1.00000 -> 0.80000

File: source/omomo_objects/tripod/tripod.urdf (robot description, URDF)
Before this commit: robot tripod, 1 links, 0 joints
Links:
- link base_link: mass 1.00000 -> 0.80000

File: source/omomo_objects/whitechair/whitechair.urdf (robot description, URDF)
Before this commit: robot whitechair, 1 links, 0 joints
Links:
- link base_link: mass 1.00000 -> 1.50000

File: source/omomo_objects/woodchair/woodchair.urdf (robot description, URDF)
Before this commit: robot woodchair, 1 links, 0 joints
Links:
- link base_link: mass 1.00000 -> 4.50000
