Commit message: updated ball mass

File: source/basketball/basketball.urdf (robot description, URDF)
Before this commit: robot basketball, 1 links, 0 joints
Links:
- link ball_link: mass 0.485 -> 0.62369

Commit message: added multi objects, upd basketball

File: source/basketball/basketball.urdf (robot description, URDF)
Before this commit: robot basketball, 1 links, 0 joints
Links:
- removed link ball_link
- added link base_link, mass 0.62369; collision sphere radius=0.12; visual sphere radius=0.12
