Commit message: decimate chair, cvx_decomp

File: source/sugar_objects/chair/chair.urdf (robot description, URDF)
Before this commit: robot chair, 1 links, 0 joints
Links:
- link base_link: geometry collision mesh filename=chair_decimated.obj; visual mesh filename=chair_decimated.obj

Commit message: refact object-model, scen gen and cvx decop add

File: source/sugar_objects/chair/chair.urdf (robot description, URDF)
Before this commit: robot chair, 1 links, 0 joints
Links:
- link base_link: geometry collision mesh filename=chair.obj; visual mesh filename=chair.obj
